File: _autosave-PPURS projekt.kicad_sch (KiCad schematic)
At the start: 26 parts, among them J2 AVR-ISP-10, J3 Barrel_Jack, SW1 SW_Push_Dual, SW2 SW_Push_Dual, U1 ATmega16A-P, U2 004-0-0053, U3 LM35-LP, U4 LCD-016N002L, Y1 8Mhz

Commit message: Add files via upload
Parts:
- C1, C2, C3, C4, C5, C6: footprint Library:CP_Radial_Tantal_D5.0mm_P5.00mmjm -> Library:CP_Radial_Tantal_D5.0mm_P5.00mmJM
- D1: footprint LED_THT:LED_D3.0mm_FlatTop -> LED_THT:LED_D5.0mm_Clear
- J3: footprint Library:BarrelJack_CUI_PJ-063AH_Horizontaljm -> Library:BarrelJack_CUI_PJ-063AH_HorizontalJM
Changed lines of the file:
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@@
       (effects (font (size 1.27 1.27)))
     )
-    (property "Footprint" "Library:CP_Radial_Tantal_D5.0mm_P5.00mmjm" (at 140.97 43.4848 0)
+    (property "Footprint" "Library:CP_Radial_Tantal_D5.0mm_P5.00mmJM" (at 140.97 43.4848 0)
       (effects (font (size 1.27 1.27)) hide)
     )
@@
       (effects (font (size 1.27 1.27)))
     )
-    (property "Footprint" "Library:CP_Radial_Tantal_D5.0mm_P5.00mmjm" (at 90.17 94.9452 0)
+    (property "Footprint" "Library:CP_Radial_Tantal_D5.0mm_P5.00mmJM" (at 90.17 94.9452 0)
       (effects (font (size 1.27 1.27)) hide)
     )
@@
       (effects (font (size 1.27 1.27)))
     )
-    (property "Footprint" "Library:CP_Radial_Tantal_D5.0mm_P5.00mmjm" (at 90.17 87.3252 0)
+    (property "Footprint" "Library:CP_Radial_Tantal_D5.0mm_P5.00mmJM" (at 90.17 87.3252 0)
       (effects (font (size 1.27 1.27)) hide)
     )
@@
       (effects (font (size 1.27 1.27)))
     )
-    (property "Footprint" "Library:BarrelJack_CUI_PJ-063AH_Horizontaljm" (at 49.53 49.276 0)
+    (property "Footprint" "Library:BarrelJack_CUI_PJ-063AH_HorizontalJM" (at 49.53 49.276 0)
       (effects (font (size 1.27 1.27)) hide)
     )
@@
       (effects (font (size 1.27 1.27)))
     )
-    (property "Footprint" "Library:CP_Radial_Tantal_D5.0mm_P5.00mmjm" (at 140.97 72.0852 0)
+    (property "Footprint" "Library:CP_Radial_Tantal_D5.0mm_P5.00mmJM" (at 140.97 72.0852 0)
       (effects (font (size 1.27 1.27)) hide)
     )
@@
       (effects (font (size 1.27 1.27)) (justify right))
     )
-    (property "Footprint" "Library:CP_Radial_Tantal_D5.0mm_P5.00mmjm" (at 108.2548 104.14 0)
+    (property "Footprint" "Library:CP_Radial_Tantal_D5.0mm_P5.00mmJM" (at 108.2548 104.14 0)
       (effects (font (size 1.27 1.27)) hide)
     )
@@
       (effects (font (size 1.27 1.27)))
     )
-    (property "Footprint" "Library:CP_Radial_Tantal_D5.0mm_P5.00mmjm" (at 261.3152 113.03 0)
+    (property "Footprint" "Library:CP_Radial_Tantal_D5.0mm_P5.00mmJM" (at 261.3152 113.03 0)
       (effects (font (size 1.27 1.27)) hide)
     )
@@
       (effects (font (size 1.27 1.27)) (justify right))
     )
-    (property "Footprint" "LED_THT:LED_D3.0mm_FlatTop" (at 162.56 133.35 0)
-      (effects (font (size 1.27 1.27)) hide)
-    )
+    (property "Footprint" "LED_THT:LED_D5.0mm_Clear" (at 162.56 133.35 0)
+      (effects (font (size 1.27 1.27)) hide)
+    )
