File: PPURS projekt.kicad_sch (KiCad schematic)
At the start: 26 parts, among them J2 AVR-ISP-10, J3 Barrel_Jack, SW1 SW_Push_Dual, SW2 SW_Push_Dual, U1 ATmega16A-P, U2 004-0-0053, U3 LM35-LP, U4 LCD-016N002L, Y1 8Mhz

Commit message: Add files via upload
Parts:
- C1, C2, C3, C4, C5, C6: footprint Library:CP_Radial_Tantal_D5.0mm_P5.00mmjm -> Library:CP_Radial_Tantal_D5.0mm_P5.00mmJM
- D1: footprint LED_THT:LED_D3.0mm_FlatTop -> LED_THT:LED_D5.0mm_Clear
- J3: footprint Library:BarrelJack_CUI_PJ-063AH_Horizontaljm -> Library:BarrelJack_CUI_PJ-063AH_HorizontalJM
Other:
- note removed: "dodati switch na buzzer"
- note removed: "mozda dodati vise ledica"
- title: (none) -> CO2 alarm sa ATmega16A-P
- moved on the sheet: BZ1, C1, C2, C3, C4, C5, C6, D1, L1, R1, R2, R3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

Commit message: pwm radi
Connections:
- net PWM: now reaches U1.17 (PD3)
- net PWM: now also U1.3 (PB2), U2.4 (PWM_1KHZ)
- no-connect marks 35 -> 32
Other:
- moved on the sheet: SW2
Changed lines of the file:
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@@
   (no_connect (at 142.24 128.27))
   (no_connect (at 199.39 111.76))
-  (no_connect (at 142.24 146.05))
   (no_connect (at 97.79 64.77))
-  (no_connect (at 261.62 46.99))
   (no_connect (at 142.24 74.93))
   (no_connect (at 219.71 121.92))
   (no_connect (at 219.71 116.84))
   (no_connect (at 231.14 52.07))
-  (no_connect (at 147.32 97.79))
+  (no_connect (at 153.67 97.79))
   (no_connect (at 142.24 156.21))
   (no_connect (at 142.24 80.01))
@@
   (no_connect (at 199.39 114.3))
   (no_connect (at 142.24 148.59))
-  (no_connect (at 142.24 97.79))
   (no_connect (at 142.24 72.39))
   (no_connect (at 142.24 77.47))
@@
   (no_connect (at 261.62 41.91))
   (no_connect (at 142.24 153.67))
-  (no_connect (at 157.48 97.79))
+  (no_connect (at 163.83 97.79))
   (wire (pts (xy 111.76 74.93) (xy 109.22 74.93))
     (stroke (width 0) (type default))
@@
     (stroke (width 0) (type default))
   )
+  (wire (pts (xy 261.62 46.99) (xy 264.16 46.99))
+    (stroke (width 0) (type default))
+  )
   (wire (pts (xy 139.7 33.02) (xy 139.7 31.75))
     (stroke (width 0) (type default))
@@
     (stroke (width 0) (type default))
   )
+  (wire (pts (xy 142.24 146.05) (xy 144.78 146.05))
+    (stroke (width 0) (type default))
+  )
   (wire (pts (xy 97.79 81.28) (xy 109.22 81.28))
     (stroke (width 0) (type default))
@@
     (stroke (width 0) (type default))
   )
-  (wire (pts (xy 165.1 99.06) (xy 165.1 92.71))
+  (wire (pts (xy 171.45 99.06) (xy 171.45 92.71))
     (stroke (width 0) (type default))
   )
@@
     (stroke (width 0) (type default))
   )
-  (wire (pts (xy 157.48 92.71) (xy 165.1 92.71))
+  (wire (pts (xy 163.83 92.71) (xy 171.45 92.71))
     (stroke (width 0) (type default))
   )
@@
     (stroke (width 0) (type default))
   )
+  (wire (pts (xy 144.78 97.79) (xy 142.24 97.79))
+    (stroke (width 0) (type default))
+  )
   (wire (pts (xy 222.25 106.68) (xy 219.71 106.68))
     (stroke (width 0) (type default))
@@
     (stroke (width 0) (type default))
   )
-  (wire (pts (xy 142.24 92.71) (xy 147.32 92.71))
+  (wire (pts (xy 142.24 92.71) (xy 153.67 92.71))
     (stroke (width 0) (type default))
   )
@@
     (effects (font (size 1.27 1.27)) (justify left bottom))
   )
+  (label "PWM" (at 144.78 146.05 0) (fields_autoplaced)
+    (effects (font (size 1.27 1.27)) (justify left bottom))
+  )
   (label "PC3" (at 144.78 123.19 0) (fields_autoplaced)
     (effects (font (size 1.27 1.27)) (justify left bottom))
@@
     (effects (font (size 1.27 1.27)) (justify left bottom))
   )
+  (label "PWM" (at 264.16 46.99 0) (fields_autoplaced)
+    (effects (font (size 1.27 1.27)) (justify left bottom))
+  )
   (label "PC0" (at 194.31 121.92 0) (fields_autoplaced)
     (effects (font (size 1.27 1.27)) (justify left bottom))
@@
   )
   (label "RESET" (at 66.04 107.95 0) (fields_autoplaced)
+    (effects (font (size 1.27 1.27)) (justify left bottom))
+  )
+  (label "PWM" (at 144.78 97.79 0) (fields_autoplaced)
     (effects (font (size 1.27 1.27)) (justify left bottom))
   )
@@
     )
   )
-  (symbol (lib_id "power:Earth") (at 165.1 99.06 0) (unit 1)
-    (in_bom yes) (on_board yes) (dnp no) (fields_autoplaced)
-    (property "Reference" "#PWR027" (at 165.1 105.41 0)
-      (effects (font (size 1.27 1.27)) hide)
-    )
-    (property "Value" "Earth" (at 165.1 102.87 0)
-      (effects (font (size 1.27 1.27)) hide)
-    )
-    (property "Footprint" "" (at 165.1 99.06 0)
-      (effects (font (size 1.27 1.27)) hide)
-    )
-    (property "Datasheet" "~" (at 165.1 99.06 0)
+  (symbol (lib_id "power:Earth") (at 171.45 99.06 0) (unit 1)
+    (in_bom yes) (on_board yes) (dnp no) (fields_autoplaced)
+    (property "Reference" "#PWR027" (at 171.45 105.41 0)
+      (effects (font (size 1.27 1.27)) hide)
+    )
+    (property "Value" "Earth" (at 171.45 102.87 0)
+      (effects (font (size 1.27 1.27)) hide)
+    )
+    (property "Footprint" "" (at 171.45 99.06 0)
+      (effects (font (size 1.27 1.27)) hide)
+    )
+    (property "Datasheet" "~" (at 171.45 99.06 0)
       (effects (font (size 1.27 1.27)) hide)
     )
@@
     )
   )
-  (symbol (lib_id "Switch:SW_Push_Dual") (at 152.4 92.71 0) (unit 1)
-    (in_bom yes) (on_board yes) (dnp no) (fields_autoplaced)
-    (property "Reference" "SW2" (at 152.4 86.36 0)
-      (effects (font (size 1.27 1.27)))
-    )
-    (property "Value" "SW_Push_Dual" (at 152.4 88.9 0)
-      (effects (font (size 1.27 1.27)))
-    )
-    (property "Footprint" "Button_Switch_THT:SW_PUSH_6mm_H7.3mm" (at 152.4 87.63 0)
-      (effects (font (size 1.27 1.27)) hide)
-    )
-    (property "Datasheet" "~" (at 152.4 87.63 0)
-      (effects (font (size 1.27 1.27)) hide)
-    )
+  (symbol (lib_id "Switch:SW_Push_Dual") (at 158.75 92.71 0) (unit 1)
+    (in_bom yes) (on_board yes) (dnp no) (fields_autoplaced)
+    (property "Reference" "SW2" (at 158.75 86.36 0)
+      (effects (font (size 1.27 1.27)))
+    )
+    (property "Value" "SW_Push_Dual" (at 158.75 88.9 0)
+      (effects (font (size 1.27 1.27)))
+    )
+    (property "Footprint" "Button_Switch_THT:SW_PUSH_6mm_H7.3mm" (at 158.75 87.63 0)
+      (effects (font (size 1.27 1.27)) hide)
+    )
+    (property "Datasheet" "~" (at 158.75 87.63 0)
+      (effects (font (size 1.27 1.27)) hide)
+    )
